File: pcb/TaikoDrum.kicad_pcb (KiCad board)
At the start: 2 copper layers, 50 x 45 mm, 34 parts, among them J1 USB_B_Micro, J2 Conn_02x04_Odd_Even, U1 STM32F103C8Tx, U3 LM358, U4 LM3940IMPX-3.3_NOPB, Y1 8Mhz

Commit message: Fixed the D+ line. the PCB schematic and layout is now 100% fully workable design. Fixed the button connection to be compatible with most generic tactile switches.
Parts:
- moved R3 7.30 mm to (106.7, 136.8), turned to 180 degrees
- moved RESET1 1.17 mm to (85.8, 129.0), turned to 0 degrees
Connections:
- J1 pad 2: D- -> Net-(J1-D-)
- J1 pad 3: D+ -> Net-(J1-D+)
- R1 pad 1: D+ -> Net-(J1-D+)
- R2 pad 1: D- -> Net-(J1-D-)
- R3 pad 1: GND -> D+
- R3 pad 2: D- -> +5V
- RESET1 pad 2: RST -> GND
- RESET1 pad 3: GND -> RST
Routing:
- net D-: track 18.7 -> 6.39 mm
- net Net-(J1-D-): track 0.00 -> 9.87 mm
- net RST: track 40.2 -> 42.2 mm
- net D+: track 16.3 -> 17.3 mm
